File: cameras/ups/camera ups/camera ups.kicad_sch (KiCad schematic)
At the start: 14 parts, among them J1 COMPUTER_POWER_BUTTON, J2 VIDEO_SYSTEM_POWER_OUT, K1 RT42xAxx

Commit message: camera ups: upgrade kicad
Parts:
- added Q1: Q_PMOS_DGS, symbol Device:Q_PMOS_DGS
- added Q2: NPN, symbol Simulation_SPICE:NPN
- added R4: 100k, symbol Device:R
- added R5, R6: 10k, symbol Device:R
- added U1: CD4541BE, Package_DIP:DIP-14_W7.62mm, symbol Timer:CD4541BE
Connections:
- net GND: now also Q2.3 (E), U1.7 (V_{SS})
- net V_CAR_BATTERY: now also R5.1
- net V_UPS: now also Q1.1 (D), R4.1; no longer K1.12
- net POWER_OUT: now reaches C3.1, F1.1, K1.11
- net POWER_OUT: now also U1.14 (V_{DD})
- new net: Q2.2 (B), R5.2, R6.2
- new net: R6.1, U1.8 (OUTPUT/Q)
- new net: K1.12, Q1.3 (S)
- new net UPS_OFF: Q1.2 (G), Q2.1 (C), R4.2
